Commit message: start attempting to add mast and camera

File: husky_custom_description/urdf/custom_description.urdf.xacro (robot description, xacro)
@@ -27,6 +27,10 @@
   <xacro:include filename="$(find husky_description)/urdf/husky.urdf.xacro" />
   <xacro:husky_robot />
-  <!-- Insert customization below, sample provided: -->
-  <link name="bowler_link">
+  <xacro:include filename="$(find husky_custom_description)/urdf/test_mast.urdf.xacro" />
+  <xacro:test_mast />
+  <!-- xacro:include filename="$(find husky_custom_description)/urdf/test_hat.urdf.xacro" />
+  <xacro:test_hat / -->
+ <!-- Insert customization below, sample provided: -->
+  <!-- link name="bowler_link">
     <visual>
       <geometry>
@@ -45,4 +49,4 @@
     <child link="bowler_link" />
     <origin xyz="0.1 -0.1 0" rpy="0 0 0.5" />
-  </joint>
+  </joint -->
 </robot>

Commit message: get a (barely) working mast on the vehicle with a single camera. All the physics values are completely bogus and control parameters are copy-paste, but it works well enough for an image to show up

File: husky_custom_description/urdf/custom_description.urdf.xacro (robot description, xacro)
@@ -27,6 +27,4 @@
   <xacro:include filename="$(find husky_description)/urdf/husky.urdf.xacro" />
   <xacro:husky_robot />
-  <xacro:include filename="$(find husky_custom_description)/urdf/test_mast.urdf.xacro" />
-  <xacro:test_mast />
   <!-- xacro:include filename="$(find husky_custom_description)/urdf/test_hat.urdf.xacro" />
   <xacro:test_hat / -->
@@ -50,3 +48,5 @@
     <origin xyz="0.1 -0.1 0" rpy="0 0 0.5" />
   </joint -->
+  <!-- xacro:include filename="$(find husky_custom_description)/urdf/test_mast.urdf.xacro" />
+  <xacro:test_mast / -->
 </robot>

File: husky_custom_description/urdf/test_mast.urdf.xacro (robot description, xacro)
@@ -1,4 +1,28 @@
 <?xml version="1.0"?>
 <robot xmlns:xacro="http://ros.org/wiki/xacro" name="test_mast">
+  <material name="Black">
+    <color rgba="0.0 0.0 0.0 1.0"/>
+  </material>
+  <material name="Blue">
+    <color rgba="0.0 0.0 0.8 1.0"/>
+  </material>
+  <material name="Green">
+    <color rgba="0.0 0.8 0.0 1.0"/>
+  </material>
+  <material name="Grey">
+    <color rgba="0.2 0.2 0.2 1.0"/>
+  </material>
+  <material name="Orange">
+    <color rgba="${255/255} ${108/255} ${10/255} 1.0"/>
+  </material>
+  <material name="Brown">
+    <color rgba="${222/255} ${207/255} ${195/255} 1.0"/>
+  </material>
+  <material name="Red">
+    <color rgba="0.8 0.0 0.0 1.0"/>
+  </material>
+  <material name="White">
+    <color rgba="1.0 1.0 1.0 1.0"/>
+  </material>
   <xacro:property name="mast_ht" value="1.6" />
   <xacro:property name="mast_h2" value="0.8" />
@@ -16,12 +40,15 @@
         <box size="0.05 0.05 ${mast_ht}"/>
       </geometry>
-      <material name="orange"/>
+      <material name="White"/>
     </visual>
     <inertial>
       <origin rpy="0 0 0" xyz="0 0 ${mast_h2}"/>
-      <mass value="1"/>
-      <inertia ixx="1.0" ixy="0.0" ixz="0.0" iyy="1.0" iyz="0.0" izz="1.0"/>
-    </inertial>
-  </link>
+      <mass value="0.2"/>
+      <inertia ixx="0.1" ixy="0.0" ixz="0.0" iyy="0.1" iyz="0.0" izz="0.1"/>
+    </inertial>
+  </link>
+  <gazebo reference="mast_link">
+    <material>Gazebo/White</material>
+  </gazebo>
   <joint name="mast_joint" type="fixed">
     <parent link="base_link"/>
@@ -42,18 +69,32 @@
         <box size="0.1 0.1 0.2"/>
       </geometry>
-      <material name="orange"/>
-    </visual>
-    <inertial>
-      <origin rpy="0 0 0" xyz="0 0 0.1"/>
-      <mass value="0.2"/>
-      <inertia ixx="1.0" ixy="0.0" ixz="0.0" iyy="1.0" iyz="0.0" izz="1.0"/>
-    </inertial>
-  </link>
-  <joint name="pan_joint" type="fixed">
+      <material name="Blue"/>
+    </visual>
+    <inertial>
+      <origin rpy="0 0 0" xyz="0 0 0.1"/>
+      <mass value="0.1"/>
+      <inertia ixx="0.1" ixy="0.0" ixz="0.0" iyy="0.1" iyz="0.0" izz="0.1"/>
+    </inertial>
+  </link>
+  <gazebo reference="pan_link">
+    <material>Gazebo/Blue</material>
+  </gazebo>
+  <joint name="pan_joint" type="revolute">
     <parent link="mast_link"/>
     <child link="pan_link"/>
     <origin xyz="0 0 ${mast_ht}" rpy="0 0 0" />
     <axis xyz="0 0 1"/>
-  </joint>
+    <limit lower="${-2.0 * pi}" upper="${2.0 * pi}" effort="150.0" velocity="3.15"/>
+  </joint>
+  <transmission name="pan_transmission">
+    <type>transmission_interface/SimpleTransmission</type>
+    <joint name="pan_joint">
+      <hardwareInterface>EffortJointInterface</hardwareInterface>
+    </joint>
+    <actuator name="pan_motor">
+      <hardwareInterface>EffortJointInterface</hardwareInterface>
+      <mechanicalReduction>1</mechanicalReduction>
+    </actuator>
+  </transmission>
   <link name="tilt_link">
     <collision>
@@ -68,12 +109,15 @@
         <box size="0.1 0.1 0.2"/>
       </geometry>
-      <material name="orange"/>
-    </visual>
-    <inertial>
-      <origin rpy="0 0 0" xyz="0 0 0.1"/>
-      <mass value="0.2"/>
-      <inertia ixx="1.0" ixy="0.0" ixz="0.0" iyy="1.0" iyz="0.0" izz="1.0"/>
-    </inertial>
-  </link>
+      <material name="Green"/>
+    </visual>
+    <inertial>
+      <origin rpy="0 0 0" xyz="0 0 0.1"/>
+      <mass value="0.1"/>
+      <inertia ixx="0.1" ixy="0.0" ixz="0.0" iyy="0.1" iyz="0.0" izz="0.1"/>
+    </inertial>
+  </link>
+  <gazebo reference="tilt_link">
+    <material>Gazebo/Green</material>
+  </gazebo>
   <joint name="tilt_joint" type="revolute">
     <parent link="pan_link"/>
@@ -83,4 +127,14 @@
     <limit lower="${-2.0 * pi}" upper="${2.0 * pi}" effort="150.0" velocity="3.15"/>
   </joint>
+  <transmission name="tilt_transmission">
+    <type>transmission_interface/SimpleTransmission</type>
+    <joint name="tilt_joint">
+      <hardwareInterface>EffortJointInterface</hardwareInterface>
+    </joint>
+    <actuator name="tilt_motor">
+      <hardwareInterface>EffortJointInterface</hardwareInterface>
+      <mechanicalReduction>1</mechanicalReduction>
+    </actuator>
+  </transmission>
   <link name="camera_link">
     <collision>
@@ -95,19 +149,14 @@
         <box size="0.1 0.1 0.1"/>
       </geometry>
-      <material name="red"/>
-    </visual>
-    <inertial>
-      <mass value="0.1" />
+      <material name="Red"/>
+    </visual>
+    <inertial>
+      <mass value="0.05" />
       <origin xyz="0 0 0" rpy="0 0 0"/>
       <inertia ixx="0.1" ixy="0" ixz="0" iyy="0.1" iyz="0" izz="0.1" />
     </inertial>
   </link>
-  <joint name="camera_joint" type="fixed">
-    <axis xyz="0 1 0" />
-    <origin xyz="0.1 0 0" rpy="0 0 0"/>
-    <parent link="tilt_link"/>
-    <child link="camera_link"/>
-  </joint>
   <gazebo reference="camera_link">
+    <material>Gazebo/Red</material>
     <sensor type="camera" name="camera1">
       <update_rate>30.0</update_rate>
@@ -145,4 +194,10 @@
     </sensor>
   </gazebo>
+  <joint name="camera_joint" type="fixed">
+    <axis xyz="0 1 0" />
+    <origin xyz="0.1 0 0.2" rpy="0 0 0"/>
+    <parent link="tilt_link"/>
+    <child link="camera_link"/>
+  </joint>
   </xacro:macro>
 </robot>
