Commit message: add a launch file that starts rapid-ros bridge

File: husky_custom_description/urdf/test_mast.urdf.xacro (robot description, xacro)
@@ -27,4 +27,6 @@
   <xacro:property name="mast_ht" value="1.6" />
   <xacro:property name="mast_h2" value="0.8" />
+  <xacro:property name="Camera01Name"       value="NavCamLeft" />
+  <xacro:property name="Camera01UpdateRate" value="0.5" />
   <xacro:macro name="test_mast">
   <link name="mast_link">
@@ -137,5 +139,5 @@
     </actuator>
   </transmission>
-  <link name="camera_link">
+  <link name="${Camera01Name}_link">
     <collision>
       <origin xyz="0 0 0" rpy="0 0 0"/>
@@ -157,8 +159,8 @@
     </inertial>
   </link>
-  <gazebo reference="camera_link">
+  <gazebo reference="${Camera01Name}_link">
     <material>Gazebo/Red</material>
-    <sensor type="camera" name="camera1">
-      <update_rate>30.0</update_rate>
+    <sensor type="camera" name="${Camera01Name}">
+      <update_rate>${Camera01UpdateRate}</update_rate>
       <camera name="head">
         <horizontal_fov>1.3962634</horizontal_fov>
@@ -181,8 +183,8 @@
         <alwaysOn>true</alwaysOn>
         <updateRate>0.0</updateRate>
-        <cameraName>mast/camera1</cameraName>
+        <cameraName>cameras/${Camera01Name}</cameraName>
         <imageTopicName>image_raw</imageTopicName>
         <cameraInfoTopicName>camera_info</cameraInfoTopicName>
-        <frameName>camera_link</frameName>
+        <frameName>${Camera01Name}_link</frameName>
         <hackBaseline>0.07</hackBaseline>
         <distortionK1>0.0</distortionK1>
@@ -198,5 +200,5 @@
     <origin xyz="0.1 0 0.2" rpy="0 0 0"/>
     <parent link="tilt_link"/>
-    <child link="camera_link"/>
+    <child link="${Camera01Name}_link"/>
   </joint>
   </xacro:macro>

Commit message: reduce limits on pan tilt

File: husky_custom_description/urdf/test_mast.urdf.xacro (robot description, xacro)
@@ -28,5 +28,6 @@
   <xacro:property name="mast_h2" value="0.8" />
   <xacro:property name="Camera01Name"       value="NavCamLeft" />
-  <xacro:property name="Camera01UpdateRate" value="0.5" />
+  <!-- xacro:property name="Camera01UpdateRate" value="0.5" / -->
+  <xacro:property name="Camera01UpdateRate" value="10" />
   <xacro:macro name="test_mast">
   <link name="mast_link">
@@ -87,5 +88,5 @@
     <origin xyz="0 0 ${mast_ht}" rpy="0 0 0" />
     <axis xyz="0 0 1"/>
-    <limit lower="${-2.0 * pi}" upper="${2.0 * pi}" effort="150.0" velocity="3.15"/>
+    <limit lower="${-1.0 * pi}" upper="${1.0 * pi}" effort="150.0" velocity="3.15"/>
   </joint>
   <transmission name="pan_transmission">
@@ -127,5 +128,5 @@
     <origin xyz="0 0 0.2" rpy="0 0.2 0" />
     <axis xyz="0 1 0"/>
-    <limit lower="${-2.0 * pi}" upper="${2.0 * pi}" effort="150.0" velocity="3.15"/>
+    <limit lower="${-1.0 * pi}" upper="${1.0 * pi}" effort="150.0" velocity="3.15"/>
   </joint>
   <transmission name="tilt_transmission">
