Commit message: add references to Mikes planners, but dont enable by default. Attempt to get shaders working in Ogre material, but it does not seem to work

File: husky_custom_description/urdf/stereo_test_mast.urdf.xacro (robot description, xacro)
@@ -28,5 +28,5 @@
   <xacro:property name="mast_h2" value="0.8" />
   <xacro:property name="Camera01Name"       value="NavCamStereo" />
-  <xacro:property name="Camera01UpdateRate" value="30" />
+  <xacro:property name="Camera01UpdateRate" value="1" />
   <xacro:property name="camera_baseline"      value="0.50" />
   <xacro:macro name="stereo_test_mast">

Commit message: put reasonable limits on pan/tilt and slow down gimbal motors

File: husky_custom_description/urdf/stereo_test_mast.urdf.xacro (robot description, xacro)
@@ -88,5 +88,5 @@
     <origin xyz="0 0 ${mast_ht}" rpy="0 0 0" />
     <axis xyz="0 0 1"/>
-    <limit lower="${-2.1 * pi}" upper="${2.1 * pi}" effort="150.0" velocity="3.15"/>
+    <limit lower="${-1.0 * pi}" upper="${1.0 * pi}" effort="8.0" velocity="0.001"/>
   </joint>
   <transmission name="pan_transmission">
@@ -128,5 +128,5 @@
     <origin xyz="0 0 0.2" rpy="0 0.2 0" />
     <axis xyz="0 1 0"/>
-    <limit lower="${-2.1 * pi}" upper="${2.1 * pi}" effort="150.0" velocity="3.15"/>
+    <limit lower="-0.1" upper="1.0" effort="2.0" velocity="0.001"/>
   </joint>
   <transmission name="tilt_transmission">

Commit message: add better inertial matrix for mast

File: husky_custom_description/urdf/stereo_test_mast.urdf.xacro (robot description, xacro)
@@ -48,5 +48,9 @@
       <origin rpy="0 0 0" xyz="0 0 ${mast_h2}"/>
       <mass value="0.2"/>
-      <inertia ixx="0.1" ixy="0.0" ixz="0.0" iyy="0.1" iyz="0.0" izz="0.1"/>
+      <!-- inertia ixx="0.01" ixy="0.0" ixz="0.0" iyy="0.01" iyz="0.0" izz="0.01"/ -->
+      <inertia
+          ixx="${0.2 / 12.0 * (0.05*0.05 + mast_ht*mast_ht)}" ixy="0.0" ixz="0.0"
+          iyy="${0.2 / 12.0 * (mast_ht*mast_ht + 0.05*0.05)}" iyz="0.0"
+          izz="${0.2 / 12.0 * (0.05*0.05 + 0.05*0.05)}"/>
     </inertial>
   </link>
@@ -77,5 +81,9 @@
       <origin rpy="0 0 0" xyz="0 0 0.1"/>
       <mass value="0.1"/>
-      <inertia ixx="0.1" ixy="0.0" ixz="0.0" iyy="0.1" iyz="0.0" izz="0.1"/>
+      <!-- inertia ixx="0.1" ixy="0.0" ixz="0.0" iyy="0.1" iyz="0.0" izz="0.1"/ -->
+      <inertia
+          ixx="${0.1 / 12.0 * (0.1*0.1 + 0.2*0.2)}" ixy="0.0" ixz="0.0"
+          iyy="${0.1 / 12.0 * (0.2*0.2 + 0.1*0.1)}" iyz="0.0"
+          izz="${0.1 / 12.0 * (0.1*0.1 + 0.1*0.1)}"/>
     </inertial>
   </link>
@@ -117,5 +125,15 @@
       <origin rpy="0 0 0" xyz="0 0 0.1"/>
       <mass value="0.1"/>
-      <inertia ixx="0.1" ixy="0.0" ixz="0.0" iyy="0.1" iyz="0.0" izz="0.1"/>
+      <!-- inertia ixx="0.1" ixy="0.0" ixz="0.0" iyy="0.1" iyz="0.0" izz="0.1"/ -->
+      <!-- see https://github.com/ros-simulation/gazebo_ros_demos/blob/master/rrbot_description/urdf/rrbot.xacro for box formula -->
+      <!-- https://en.wikipedia.org/wiki/List_of_moments_of_inertia -->
+      <!-- inertia
+          ixx="${mass / 12.0 * (depth*depth + height*height)}" ixy="0.0" ixz="0.0"
+          iyy="${mass / 12.0 * (height*height + width*width)}" iyz="0.0"
+          izz="${mass / 12.0 * (depth*depth + width*width)}"/ -->
+     <inertia
+          ixx="${0.1 / 12.0 * (0.1*0.1 + 0.2*0.2)}" ixy="0.0" ixz="0.0"
+          iyy="${0.1 / 12.0 * (0.2*0.2 + 0.1*0.1)}" iyz="0.0"
+          izz="${0.1 / 12.0 * (0.1*0.1 + 0.1*0.1)}"/>
     </inertial>
   </link>
@@ -172,5 +190,13 @@
       <origin xyz="0 0 0" rpy="0 0 0"/>
       <inertia ixx="0.1" ixy="0" ixz="0" iyy="0.1" iyz="0" izz="0.1" />
-    </inertial>
+      <!-- inertia
+          ixx="${mass / 12.0 * (depth*depth + height*height)}" ixy="0.0" ixz="0.0"
+          iyy="${mass / 12.0 * (height*height + width*width)}" iyz="0.0"
+          izz="${mass / 12.0 * (depth*depth + width*width)}"/ -->
+      <!-- inertia
+          ixx="${0.05 / 12.0 * (0.1*0.1 + 0.1*0.1)}" ixy="0.0" ixz="0.0"
+          iyy="${0.05 / 12.0 * (0.1*0.1 + camera_baseline*camera_baseline)}" iyz="0.0"
+          izz="${0.05 / 12.0 * (0.1*0.1 + camera_baseline*camera_baseline)}"/-->
+   </inertial>
   </link>
   <gazebo reference="${Camera01Name}_link">

Commit message: adding left & right camera frames

File: husky_custom_description/urdf/stereo_test_mast.urdf.xacro (robot description, xacro)
@@ -165,11 +165,11 @@
       </geometry>
     </collision>
-    <visual>
-      <origin xyz="0 0 0"  rpy="0 0 0"/>
-      <geometry>
-        <box size="0.025 ${camera_baseline} 0.025"/>
-      </geometry>
-      <material name="Red"/>
-    </visual>
+      <visual>
+        <origin xyz="0 0 0"  rpy="0 0 0"/>
+        <geometry>
+          <box size="0.025 ${camera_baseline} 0.025"/>
+        </geometry>
+        <material name="Red"/>
+      </visual>
     <visual>
       <origin xyz="0 ${camera_baseline/2} 0"  rpy="0 0 0"/>
@@ -205,20 +205,20 @@
       <update_rate>${Camera01UpdateRate}</update_rate>
       <camera name="left">
-        <pose>0 ${camera_baseline/2} 0 0 0 0</pose>
-        <horizontal_fov>1.3962634</horizontal_fov>
-        <image>
-          <width>800</width>
-          <height>800</height>
-          <format>R8G8B8</format>
-        </image>
-        <clip>
-          <near>0.02</near>
-          <far>300</far>
-        </clip>
-        <noise>
-          <type>gaussian</type>
-          <mean>0.0</mean>
-          <stddev>0.007</stddev>
-        </noise>
+          <pose>0 ${camera_baseline/2} 0 0 0 0</pose>
+          <horizontal_fov>1.3962634</horizontal_fov>
+          <image>
+            <width>800</width>
+            <height>800</height>
+            <format>R8G8B8</format>
+          </image>
+          <clip>
+            <near>0.02</near>
+            <far>300</far>
+          </clip>
+          <noise>
+            <type>gaussian</type>
+            <mean>0.0</mean>
+            <stddev>0.007</stddev>
+          </noise>
       </camera>
       <camera name="right">
@@ -262,4 +262,20 @@
     <child link="${Camera01Name}_link"/>
   </joint>
+  <gazebo reference="${Camera01Name}Left_link"/>
+  <link name="${Camera01Name}Left_link"/>
+  <joint name="leftCamera_joint" type="fixed">
+    <axis xyz="0 1 0" />
+    <origin xyz="0.0 ${camera_baseline/2} 0.0" rpy="0 0 0"/>
+    <parent link="${Camera01Name}_link"/>
+    <child link="${Camera01Name}Left_link"/>
+  </joint>
+  <gazebo reference="${Camera01Name}Right_link"/>
+  <link name="${Camera01Name}Right_link"/>
+  <joint name="rightCamera_joint" type="fixed">
+    <axis xyz="0 1 0" />
+    <origin xyz="0.0 -${camera_baseline/2} 0.0" rpy="0 0 0"/>
+    <parent link="${Camera01Name}_link"/>
+    <child link="${Camera01Name}Right_link"/>
+  </joint>
   </xacro:macro>
 </robot>

Commit message: Transforming coordinate for left & right cameras to required format:   X right, Y down Z forward

File: husky_custom_description/urdf/stereo_test_mast.urdf.xacro (robot description, xacro)
@@ -266,5 +266,5 @@
   <joint name="leftCamera_joint" type="fixed">
     <axis xyz="0 1 0" />
-    <origin xyz="0.0 ${camera_baseline/2} 0.0" rpy="0 0 0"/>
+    <origin xyz="0.0 ${camera_baseline/2} 0.0" rpy="-${pi/2.0} 0 -${pi/2.0}"/>
     <parent link="${Camera01Name}_link"/>
     <child link="${Camera01Name}Left_link"/>
@@ -274,5 +274,5 @@
   <joint name="rightCamera_joint" type="fixed">
     <axis xyz="0 1 0" />
-    <origin xyz="0.0 -${camera_baseline/2} 0.0" rpy="0 0 0"/>
+    <origin xyz="0.0 -${camera_baseline/2} 0.0" rpy="-${pi/2.0} 0 -${pi/2.0}"/>
     <parent link="${Camera01Name}_link"/>
     <child link="${Camera01Name}Right_link"/>
